File: PCB/Carte Mere/Carte Mere.kicad_sch (KiCad schematic)
At the start: 2 parts

Commit message: test
Parts:
- added D? (x4): D, symbol Device:D
Other:
- moved on the sheet: U?
Changed lines of the file:
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@@
 (kicad_sch (version 20211123) (generator eeschema)
   (paper "USLetter")
-  (symbol (lib_id "Driver_Motor:ZXBM5210-S") (at 130.81 49.022 0) (unit 1)
+  (symbol (lib_id "Device:D") (at 116.586 52.832 180) (unit 1)
+    (in_bom yes) (on_board yes)
+    (property "Reference" "D?" (id 0) (at 117.094 48.768 0))
+    (property "Value" "D" (id 1) (at 116.586 50.546 0))
+    (property "Footprint" "" (id 2) (at 116.586 52.832 0)
+      (effects (font (size 1.27 1.27)) hide)
+    )
+    (property "Datasheet" "~" (id 3) (at 116.586 52.832 0)
+      (effects (font (size 1.27 1.27)) hide)
+    )
+    (pin "1")
+    (pin "2")
+  )
+  (symbol (lib_id "Device:D") (at 125.984 52.832 180) (unit 1)
+    (in_bom yes) (on_board yes)
+    (property "Reference" "D?" (id 0) (at 126.492 48.768 0))
+    (property "Value" "D" (id 1) (at 125.984 50.546 0))
+    (property "Footprint" "" (id 2) (at 125.984 52.832 0)
+      (effects (font (size 1.27 1.27)) hide)
+    )
+    (property "Datasheet" "~" (id 3) (at 125.984 52.832 0)
+      (effects (font (size 1.27 1.27)) hide)
+    )
+    (pin "1")
+    (pin "2")
+  )
+  (symbol (lib_id "Device:D") (at 126.492 44.704 180) (unit 1)
+    (in_bom yes) (on_board yes)
+    (property "Reference" "D?" (id 0) (at 127 40.64 0))
+    (property "Value" "D" (id 1) (at 126.492 42.418 0))
+    (property "Footprint" "" (id 2) (at 126.492 44.704 0)
+      (effects (font (size 1.27 1.27)) hide)
+    )
+    (property "Datasheet" "~" (id 3) (at 126.492 44.704 0)
+      (effects (font (size 1.27 1.27)) hide)
+    )
+    (pin "1")
+    (pin "2")
+  )
+  (symbol (lib_id "Driver_Motor:ZXBM5210-S") (at 157.226 50.038 0) (unit 1)
     (in_bom yes) (on_board yes) (fields_autoplaced)
-    (property "Reference" "U?" (id 0) (at 132.8294 57.15 0)
+    (property "Reference" "U?" (id 0) (at 159.2454 58.166 0)
       (effects (font (size 1.27 1.27)) (justify left))
     )
-    (property "Value" "ZXBM5210-S" (id 1) (at 132.8294 59.69 0)
+    (property "Value" "ZXBM5210-S" (id 1) (at 159.2454 60.706 0)
       (effects (font (size 1.27 1.27)) (justify left))
     )
-    (property "Footprint" "Package_SO:SOIC-8_3.9x4.9mm_P1.27mm" (id 2) (at 132.08 55.372 0)
+    (property "Footprint" "Package_SO:SOIC-8_3.9x4.9mm_P1.27mm" (id 2) (at 158.496 56.388 0)
       (effects (font (size 1.27 1.27)) hide)
     )
-    (property "Datasheet" "https://www.diodes.com/assets/Datasheets/ZXBM5210.pdf" (id 3) (at 130.81 49.022 0)
+    (property "Datasheet" "https://www.diodes.com/assets/Datasheets/ZXBM5210.pdf" (id 3) (at 157.226 50.038 0)
       (effects (font (size 1.27 1.27)) hide)
     )
@@
     (pin "8")
   )
+  (symbol (lib_id "Device:D") (at 117.094 44.704 180) (unit 1)
+    (in_bom yes) (on_board yes)
+    (property "Reference" "D?" (id 0) (at 117.602 40.64 0))
+    (property "Value" "D" (id 1) (at 117.094 42.418 0))
+    (property "Footprint" "" (id 2) (at 117.094 44.704 0)
+      (effects (font (size 1.27 1.27)) hide)
+    )
+    (property "Datasheet" "~" (id 3) (at 117.094 44.704 0)
+      (effects (font (size 1.27 1.27)) hide)
+    )
+    (pin "1")
+    (pin "2")
+  )
   (sheet_instances
     (path "/" (page "1"))
   )
   (symbol_instances
+    (path "/94ff7ccf-1795-4c28-b581-f2ea7c835610"
+      (reference "D?") (unit 1) (value "D") (footprint "")
+    )
+    (path "/9851983f-a26d-497d-a5dc-46fbdc2833a9"
+      (reference "D?") (unit 1) (value "D") (footprint "")
+    )
+    (path "/9c05760e-1c55-4cc9-af2b-fa0e019403a5"
+      (reference "D?") (unit 1) (value "D") (footprint "")
+    )
+    (path "/fa68f4ce-6070-4bc3-9036-4fbcdc86d398"
+      (reference "D?") (unit 1) (value "D") (footprint "")
+    )
     (path "/a0ab7880-64b9-4d89-90ef-d0e980743707"
       (reference "U?") (unit 1) (value "ZXBM5210-S") (footprint "Package_SO:SOIC-8_3.9x4.9mm_P1.27mm")

Commit message: no message
Parts:
- removed D? (x4): D, symbol Device:D
- removed U? (x2): ZXBM5210-S, Package_SO:SOIC-8_3.9x4.9mm_P1.27mm, symbol Driver_Motor:ZXBM5210-S
Other:
- added sheet Carte Mere (untitled.kicad_sch)
Changed lines of the file:
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@@
 (kicad_sch (version 20211123) (generator eeschema)
   (paper "USLetter")
-  (symbol (lib_id "Device:D") (at 116.586 52.832 180) (unit 1)
-    (in_bom yes) (on_board yes)
-    (property "Reference" "D?" (id 0) (at 117.094 48.768 0))
-    (property "Value" "D" (id 1) (at 116.586 50.546 0))
-    (property "Footprint" "" (id 2) (at 116.586 52.832 0)
-      (effects (font (size 1.27 1.27)) hide)
+  (sheet (at 21.336 147.32) (size 80.264 48.26) (fields_autoplaced)
+    (stroke (width 0.1524) (type solid) (color 0 0 0 0))
+    (fill (color 0 0 0 0.0000))
+    (property "Sheet name" "Carte Mere" (id 0) (at 21.336 146.6084 0)
+      (effects (font (size 1.27 1.27)) (justify left bottom))
     )
-    (property "Datasheet" "~" (id 3) (at 116.586 52.832 0)
-      (effects (font (size 1.27 1.27)) hide)
+    (property "Sheet file" "untitled.kicad_sch" (id 1) (at 21.336 196.1646 0)
+      (effects (font (size 1.27 1.27)) (justify left top))
     )
-    (pin "1")
-    (pin "2")
-  )
-  (symbol (lib_id "Device:D") (at 125.984 52.832 180) (unit 1)
-    (in_bom yes) (on_board yes)
-    (property "Reference" "D?" (id 0) (at 126.492 48.768 0))
-    (property "Value" "D" (id 1) (at 125.984 50.546 0))
-    (property "Footprint" "" (id 2) (at 125.984 52.832 0)
-      (effects (font (size 1.27 1.27)) hide)
-    )
-    (property "Datasheet" "~" (id 3) (at 125.984 52.832 0)
-      (effects (font (size 1.27 1.27)) hide)
-    )
-    (pin "1")
-    (pin "2")
-  )
-  (symbol (lib_id "Device:D") (at 126.492 44.704 180) (unit 1)
-    (in_bom yes) (on_board yes)
-    (property "Reference" "D?" (id 0) (at 127 40.64 0))
-    (property "Value" "D" (id 1) (at 126.492 42.418 0))
-    (property "Footprint" "" (id 2) (at 126.492 44.704 0)
-      (effects (font (size 1.27 1.27)) hide)
-    )
-    (property "Datasheet" "~" (id 3) (at 126.492 44.704 0)
-      (effects (font (size 1.27 1.27)) hide)
-    )
-    (pin "1")
-    (pin "2")
-  )
-  (symbol (lib_id "Driver_Motor:ZXBM5210-S") (at 157.226 50.038 0) (unit 1)
-    (in_bom yes) (on_board yes) (fields_autoplaced)
-    (property "Reference" "U?" (id 0) (at 159.2454 58.166 0)
-      (effects (font (size 1.27 1.27)) (justify left))
-    )
-    (property "Value" "ZXBM5210-S" (id 1) (at 159.2454 60.706 0)
-      (effects (font (size 1.27 1.27)) (justify left))
-    )
-    (property "Footprint" "Package_SO:SOIC-8_3.9x4.9mm_P1.27mm" (id 2) (at 158.496 56.388 0)
-      (effects (font (size 1.27 1.27)) hide)
-    )
-    (property "Datasheet" "https://www.diodes.com/assets/Datasheets/ZXBM5210.pdf" (id 3) (at 157.226 50.038 0)
-      (effects (font (size 1.27 1.27)) hide)
-    )
-    (pin "1")
-    (pin "2")
-    (pin "3")
-    (pin "4")
-    (pin "5")
-    (pin "6")
-    (pin "7")
-    (pin "8")
-  )
-  (symbol (lib_id "Driver_Motor:ZXBM5210-S") (at 100.076 49.022 0) (unit 1)
-    (in_bom yes) (on_board yes) (fields_autoplaced)
-    (property "Reference" "U?" (id 0) (at 102.0954 57.15 0)
-      (effects (font (size 1.27 1.27)) (justify left))
-    )
-    (property "Value" "ZXBM5210-S" (id 1) (at 102.0954 59.69 0)
-      (effects (font (size 1.27 1.27)) (justify left))
-    )
-    (property "Footprint" "Package_SO:SOIC-8_3.9x4.9mm_P1.27mm" (id 2) (at 101.346 55.372 0)
-      (effects (font (size 1.27 1.27)) hide)
-    )
-    (property "Datasheet" "https://www.diodes.com/assets/Datasheets/ZXBM5210.pdf" (id 3) (at 100.076 49.022 0)
-      (effects (font (size 1.27 1.27)) hide)
-    )
-    (pin "1")
-    (pin "2")
-    (pin "3")
-    (pin "4")
-    (pin "5")
-    (pin "6")
-    (pin "7")
-    (pin "8")
-  )
-  (symbol (lib_id "Device:D") (at 117.094 44.704 180) (unit 1)
-    (in_bom yes) (on_board yes)
-    (property "Reference" "D?" (id 0) (at 117.602 40.64 0))
-    (property "Value" "D" (id 1) (at 117.094 42.418 0))
-    (property "Footprint" "" (id 2) (at 117.094 44.704 0)
-      (effects (font (size 1.27 1.27)) hide)
-    )
-    (property "Datasheet" "~" (id 3) (at 117.094 44.704 0)
-      (effects (font (size 1.27 1.27)) hide)
-    )
-    (pin "1")
-    (pin "2")
   )
   (sheet_instances
     (path "/" (page "1"))
+    (path "/f43f384e-6bcf-4d6c-ac65-2e849bdb75c5" (page "2"))
   )
   (symbol_instances
-    (path "/94ff7ccf-1795-4c28-b581-f2ea7c835610"
+    (path "/f43f384e-6bcf-4d6c-ac65-2e849bdb75c5/091b606b-3407-49b7-bb75-87640f1c8a39"
+      (reference "#PWR?") (unit 1) (value "GND") (footprint "")
+    )
+    (path "/f43f384e-6bcf-4d6c-ac65-2e849bdb75c5/29ff5fc2-32c3-4d84-a20d-083d7cf1e9de"
+      (reference "#PWR?") (unit 1) (value "GND") (footprint "")
+    )
+    (path "/f43f384e-6bcf-4d6c-ac65-2e849bdb75c5/3244bb61-fea4-4f7e-8fcc-4d8c3ae2ea10"
+      (reference "#PWR?") (unit 1) (value "GND") (footprint "")
+    )
+    (path "/f43f384e-6bcf-4d6c-ac65-2e849bdb75c5/52064152-4b25-4796-8ab1-2e49f3df562c"
+      (reference "#PWR?") (unit 1) (value "GND") (footprint "")
+    )
+    (path "/f43f384e-6bcf-4d6c-ac65-2e849bdb75c5/7e1e82ef-592b-4651-b93e-3f98218ff854"
+      (reference "#PWR?") (unit 1) (value "GND") (footprint "")
+    )
+    (path "/f43f384e-6bcf-4d6c-ac65-2e849bdb75c5/7e5943f9-6688-4095-8776-357143e1d703"
+      (reference "#PWR?") (unit 1) (value "GND") (footprint "")
+    )
+    (path "/f43f384e-6bcf-4d6c-ac65-2e849bdb75c5/8b550f68-7124-4893-aca9-14a3e63d5e44"
+      (reference "#PWR?") (unit 1) (value "GND") (footprint "")
+    )
+    (path "/f43f384e-6bcf-4d6c-ac65-2e849bdb75c5/ec8e706c-77ef-4c50-937e-b0055b2fef44"
+      (reference "#PWR?") (unit 1) (value "GND") (footprint "")
+    )
+    (path "/f43f384e-6bcf-4d6c-ac65-2e849bdb75c5/17ff1d15-b2c6-4754-b00c-b6562e19757a"
+      (reference "C?") (unit 1) (value "0.1uf") (footprint "")
+    )
+    (path "/f43f384e-6bcf-4d6c-ac65-2e849bdb75c5/2b1d77fe-f78d-4ff8-b505-0f28f2dbc7c6"
+      (reference "C?") (unit 1) (value "0.1uf") (footprint "")
+    )
+    (path "/f43f384e-6bcf-4d6c-ac65-2e849bdb75c5/37d837fc-0a1c-47e3-82b3-d714c000df6c"
+      (reference "C?") (unit 1) (value "0.1uf") (footprint "")
+    )
+    (path "/f43f384e-6bcf-4d6c-ac65-2e849bdb75c5/3df86da9-5e08-4334-80a3-55df1ef7e8aa"
+      (reference "C?") (unit 1) (value "10uf") (footprint "Capacitor_SMD:C_0805_2012Metric_Pad1.18x1.45mm_HandSolder")
+    )
+    (path "/f43f384e-6bcf-4d6c-ac65-2e849bdb75c5/644f2a5e-73b6-4699-9c2e-a861b88658a1"
+      (reference "C?") (unit 1) (value "10uf") (footprint "Capacitor_SMD:C_0805_2012Metric_Pad1.18x1.45mm_HandSolder")
+    )
+    (path "/f43f384e-6bcf-4d6c-ac65-2e849bdb75c5/81f7250e-df81-4533-8952-51948cdec85d"
+      (reference "C?") (unit 1) (value "10uf") (footprint "Capacitor_SMD:C_0805_2012Metric_Pad1.18x1.45mm_HandSolder")
+    )
+    (path "/f43f384e-6bcf-4d6c-ac65-2e849bdb75c5/988553e8-37e3-480b-af1c-3a142d19c33c"
+      (reference "C?") (unit 1) (value "0.1uf") (footprint "")
+    )
+    (path "/f43f384e-6bcf-4d6c-ac65-2e849bdb75c5/e4b2bdc6-b3a2-44dc-b9c9-3872d6ec7b1d"
+      (reference "C?") (unit 1) (value "0.33uf") (footprint "Capacitor_SMD:C_0805_2012Metric_Pad1.18x1.45mm_HandSolder")
+    )
+    (path "/f43f384e-6bcf-4d6c-ac65-2e849bdb75c5/02297bbb-ab4c-4b32-b01f-a1a47b5f8881"
       (reference "D?") (unit 1) (value "D") (footprint "")
     )
-    (path "/9851983f-a26d-497d-a5dc-46fbdc2833a9"
+    (path "/f43f384e-6bcf-4d6c-ac65-2e849bdb75c5/3060d34f-282b-4e2e-b643-89ff682f0aeb"
       (reference "D?") (unit 1) (value "D") (footprint "")
     )
-    (path "/9c05760e-1c55-4cc9-af2b-fa0e019403a5"
+    (path "/f43f384e-6bcf-4d6c-ac65-2e849bdb75c5/7d0f503a-f1ce-4b37-aae9-b33f9c1a865e"
       (reference "D?") (unit 1) (value "D") (footprint "")
     )
-    (path "/fa68f4ce-6070-4bc3-9036-4fbcdc86d398"
+    (path "/f43f384e-6bcf-4d6c-ac65-2e849bdb75c5/967a2466-b1b0-45d5-ab7d-44da3d0d228e"
       (reference "D?") (unit 1) (value "D") (footprint "")
     )
-    (path "/a0ab7880-64b9-4d89-90ef-d0e980743707"
+    (path "/f43f384e-6bcf-4d6c-ac65-2e849bdb75c5/8299eba0-e837-4e71-bbdf-7d14f395062c"
+      (reference "R?") (unit 1) (value "R_US") (footprint "")
+    )
+    (path "/f43f384e-6bcf-4d6c-ac65-2e849bdb75c5/b5506da1-384c-4aab-83ed-9f96813b1f5e"
+      (reference "R?") (unit 1) (value "R_US") (footprint "")
+    )
+    (path "/f43f384e-6bcf-4d6c-ac65-2e849bdb75c5/1c297131-deeb-400e-918a-e0d68f026d4d"
       (reference "U?") (unit 1) (value "ZXBM5210-S") (footprint "Package_SO:SOIC-8_3.9x4.9mm_P1.27mm")
     )
-    (path "/e891b433-8f8c-451a-9a1f-eebc6bd34030"
+    (path "/f43f384e-6bcf-4d6c-ac65-2e849bdb75c5/3dddd66b-095d-4aa4-88a9-bc08a2503519"
+      (reference "U?") (unit 1) (value "MC33269DR2-5.0G") (footprint "Package_SO:SOIC-8_3.9x4.9mm_P1.27mm")
+    )
+    (path "/f43f384e-6bcf-4d6c-ac65-2e849bdb75c5/555ab27b-a08d-42b8-9a27-64f618b56dfb"
+      (reference "U?") (unit 1) (value "LM1117-3.3") (footprint "")
+    )
+    (path "/f43f384e-6bcf-4d6c-ac65-2e849bdb75c5/f3dd25e6-a44a-416a-bd30-445c8707ad54"
       (reference "U?") (unit 1) (value "ZXBM5210-S") (footprint "Package_SO:SOIC-8_3.9x4.9mm_P1.27mm")
     )

Commit message: 1.2 PCB
Other:
- added sheet Capteur (Capteur infrarouge.kicad_sch)
