File: PCB/Carte Mere/Capteur infrarouge.kicad_sch (KiCad schematic)
At the start: 15 parts, among them J10 TRCT5000, J11 TRCT5000, J5 IR204, J6 IR204, J7 TL1838, J8 TRCT5000, J9 TRCT5000

Commit message: 1.5 PCB
Parts:
- removed J10, J11, J8, J9: TRCT5000, symbol Connector_Generic:Conn_02x02_Counter_Clockwise
- added J10, J11, J8, J9: Conn_01x04_Male, symbol Connector:Conn_01x04_Male
- added U5, U6, U7, U8: TCRT5000, symbol TCRT5000:TCRT5000
- R4: value 10kΩ -> 500Ω
- R7: value 500Ω -> 10kΩ
Connections:
- net GND: now also J10.2 (Pin_2), J11.2 (Pin_2), J8.2 (Pin_2), J9.2 (Pin_2), U5.CATH, U5.E, U6.CATH, U6.E, U7.CATH, U7.E, U8.CATH, U8.E
- net at R3.2: now also U6.A
- net at R4.2: now also U7.A
- net A0: now reaches R10.1
- net A0: now also R6.1, R7.1, R8.1, J10.4 (Pin_4), J11.4 (Pin_4), J8.4 (Pin_4), J9.4 (Pin_4), U5.COLL, U6.COLL, U7.COLL, U8.COLL
- net 5V: now reaches R10.2
- net 5V: now also R6.2, R7.2, R8.2, J10.1 (Pin_1), J11.1 (Pin_1), J8.1 (Pin_1), J9.1 (Pin_1)
- net P6: now reaches R4.1
- net P6: now also J10.3 (Pin_3)
- net P5: now reaches R3.1
- net P5: now also J9.3 (Pin_3)
- net at R5.2: now also U8.A
- net P4: now reaches R9.1
- net P4: now also J8.3 (Pin_3)
- net at R9.2: now also U5.A
- net P7: now reaches R5.1
- net P7: now also J11.3 (Pin_3)
Other:
- moved on the sheet: J5, J6, J7, R10, R9

Commit message: 1.6
Parts:
- J10: renamed from J8; footprint (none) -> Connector_PinHeader_2.54mm:PinHeader_1x04_P2.54mm_Vertical
- J11: renamed from J9; footprint (none) -> Connector_PinHeader_2.54mm:PinHeader_1x04_P2.54mm_Vertical
- J12: renamed from J10; footprint (none) -> Connector_PinHeader_2.54mm:PinHeader_1x04_P2.54mm_Vertical
- J13: renamed from J11; footprint (none) -> Connector_PinHeader_2.54mm:PinHeader_1x04_P2.54mm_Vertical
- U5, U6, U7, U8: footprint (none) -> Library:tcrt5000
- renumbered J5 to J7, J6 to J8, J7 to J9, R8 to R10, R9 to R3, R3 to R4, R4 to R5, R5 to R6, R10 to R7, R6 to R8, R7 to R9
Changed lines of the file:
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@@
   (symbol (lib_id "Device:R_Small_US") (at 244.348 66.802 90) (unit 1)
     (in_bom yes) (on_board yes)
-    (property "Reference" "R10" (id 0) (at 244.348 68.834 90))
+    (property "Reference" "R7" (id 0) (at 244.348 68.834 90))
     (property "Value" "10kΩ" (id 1) (at 244.348 70.358 90))
     (property "Footprint" "Resistor_SMD:R_0805_2012Metric_Pad1.20x1.40mm_HandSolder" (id 2) (at 244.348 66.802 0)
@@
   (symbol (lib_id "Connector:Conn_01x03_Male") (at 108.712 105.156 180) (unit 1)
     (in_bom yes) (on_board yes)
-    (property "Reference" "J7" (id 0) (at 109.982 103.886 0)
+    (property "Reference" "J9" (id 0) (at 109.982 103.886 0)
       (effects (font (size 1.27 1.27)) (justify right))
     )
@@
   (symbol (lib_id "Device:R_Small_US") (at 245.364 136.398 90) (unit 1)
     (in_bom yes) (on_board yes)
-    (property "Reference" "R8" (id 0) (at 245.364 138.43 90))
+    (property "Reference" "R10" (id 0) (at 245.364 138.43 90))
     (property "Value" "10kΩ" (id 1) (at 245.364 139.954 90))
     (property "Footprint" "Resistor_SMD:R_0805_2012Metric_Pad1.20x1.40mm_HandSolder" (id 2) (at 245.364 136.398 0)
@@
   (symbol (lib_id "Connector:Conn_01x02_Male") (at 108.712 97.79 180) (unit 1)
     (in_bom yes) (on_board yes) (fields_autoplaced)
-    (property "Reference" "J6" (id 0) (at 110.236 95.2499 0)
+    (property "Reference" "J8" (id 0) (at 110.236 95.2499 0)
       (effects (font (size 1.27 1.27)) (justify right))
     )
@@
   (symbol (lib_id "Device:R_Small_US") (at 217.17 89.916 90) (unit 1)
     (in_bom yes) (on_board yes)
-    (property "Reference" "R3" (id 0) (at 217.424 86.36 90))
+    (property "Reference" "R4" (id 0) (at 217.424 86.36 90))
     (property "Value" "500Ω" (id 1) (at 217.17 88.138 90))
     (property "Footprint" "Resistor_SMD:R_0805_2012Metric_Pad1.20x1.40mm_HandSolder" (id 2) (at 217.17 89.916 0)
@@
     (property "Reference" "U8" (id 0) (at 232.156 130.81 0))
     (property "Value" "TCRT5000" (id 1) (at 232.156 132.842 0))
-    (property "Footprint" "" (id 2) (at 232.156 138.938 0)
+    (property "Footprint" "Library:tcrt5000" (id 2) (at 232.156 138.938 0)
       (effects (font (size 1.27 1.27)) (justify left bottom) hide)
     )
@@
   (symbol (lib_id "Device:R_Small_US") (at 217.678 113.284 90) (unit 1)
     (in_bom yes) (on_board yes)
-    (property "Reference" "R4" (id 0) (at 217.932 109.728 90))
+    (property "Reference" "R5" (id 0) (at 217.932 109.728 90))
     (property "Value" "500Ω" (id 1) (at 217.678 111.506 90))
     (property "Footprint" "Resistor_SMD:R_0805_2012Metric_Pad1.20x1.40mm_HandSolder" (id 2) (at 217.678 113.284 0)
@@
   (symbol (lib_id "Connector:Conn_01x04_Male") (at 197.612 90.17 0) (unit 1)
     (in_bom yes) (on_board yes)
-    (property "Reference" "J9" (id 0) (at 200.406 83.312 0))
+    (property "Reference" "J11" (id 0) (at 200.406 83.312 0))
     (property "Value" "Conn_01x04_Male" (id 1) (at 200.406 85.09 0))
-    (property "Footprint" "" (id 2) (at 197.612 90.17 0)
+    (property "Footprint" "Connector_PinHeader_2.54mm:PinHeader_1x04_P2.54mm_Vertical" (id 2) (at 197.612 90.17 0)
       (effects (font (size 1.27 1.27)) hide)
     )
@@
     (property "Reference" "U6" (id 0) (at 231.394 84.328 0))
     (property "Value" "TCRT5000" (id 1) (at 231.394 86.36 0))
-    (property "Footprint" "" (id 2) (at 231.394 92.456 0)
+    (property "Footprint" "Library:tcrt5000" (id 2) (at 231.394 92.456 0)
       (effects (font (size 1.27 1.27)) (justify left bottom) hide)
     )
@@
   (symbol (lib_id "Connector:Conn_01x04_Male") (at 197.358 67.056 0) (unit 1)
     (in_bom yes) (on_board yes)
-    (property "Reference" "J8" (id 0) (at 200.152 60.198 0))
+    (property "Reference" "J10" (id 0) (at 200.152 60.198 0))
     (property "Value" "Conn_01x04_Male" (id 1) (at 200.152 61.976 0))
-    (property "Footprint" "" (id 2) (at 197.358 67.056 0)
+    (property "Footprint" "Connector_PinHeader_2.54mm:PinHeader_1x04_P2.54mm_Vertical" (id 2) (at 197.358 67.056 0)
       (effects (font (size 1.27 1.27)) hide)
     )
@@
   (symbol (lib_id "Device:R_Small_US") (at 217.932 136.398 90) (unit 1)
     (in_bom yes) (on_board yes)
-    (property "Reference" "R5" (id 0) (at 218.186 132.842 90))
+    (property "Reference" "R6" (id 0) (at 218.186 132.842 90))
     (property "Value" "500Ω" (id 1) (at 217.932 134.62 90))
     (property "Footprint" "Resistor_SMD:R_0805_2012Metric_Pad1.20x1.40mm_HandSolder" (id 2) (at 217.932 136.398 0)
@@
   (symbol (lib_id "Connector:Conn_01x04_Male") (at 198.374 136.652 0) (unit 1)
     (in_bom yes) (on_board yes)
-    (property "Reference" "J11" (id 0) (at 201.168 129.794 0))
+    (property "Reference" "J13" (id 0) (at 201.168 129.794 0))
     (property "Value" "Conn_01x04_Male" (id 1) (at 201.168 131.572 0))
-    (property "Footprint" "" (id 2) (at 198.374 136.652 0)
+    (property "Footprint" "Connector_PinHeader_2.54mm:PinHeader_1x04_P2.54mm_Vertical" (id 2) (at 198.374 136.652 0)
       (effects (font (size 1.27 1.27)) hide)
     )
@@
   (symbol (lib_id "Connector:Conn_01x02_Male") (at 108.712 90.424 180) (unit 1)
     (in_bom yes) (on_board yes) (fields_autoplaced)
-    (property "Reference" "J5" (id 0) (at 110.236 87.8839 0)
+    (property "Reference" "J7" (id 0) (at 110.236 87.8839 0)
       (effects (font (size 1.27 1.27)) (justify right))
     )
@@
   (symbol (lib_id "Device:R_Small_US") (at 244.602 89.916 90) (unit 1)
     (in_bom yes) (on_board yes)
-    (property "Reference" "R6" (id 0) (at 244.602 91.948 90))
+    (property "Reference" "R8" (id 0) (at 244.602 91.948 90))
     (property "Value" "10kΩ" (id 1) (at 244.602 93.472 90))
     (property "Footprint" "Resistor_SMD:R_0805_2012Metric_Pad1.20x1.40mm_HandSolder" (id 2) (at 244.602 89.916 0)
@@
   (symbol (lib_id "Device:R_Small_US") (at 216.916 66.802 90) (unit 1)
     (in_bom yes) (on_board yes)
-    (property "Reference" "R9" (id 0) (at 217.17 63.246 90))
+    (property "Reference" "R3" (id 0) (at 217.17 63.246 90))
     (property "Value" "500Ω" (id 1) (at 216.916 65.024 90))
     (property "Footprint" "Resistor_SMD:R_0805_2012Metric_Pad1.20x1.40mm_HandSolder" (id 2) (at 216.916 66.802 0)
@@
     (property "Reference" "U5" (id 0) (at 231.14 61.214 0))
     (property "Value" "TCRT5000" (id 1) (at 231.14 63.246 0))
-    (property "Footprint" "" (id 2) (at 231.14 69.342 0)
+    (property "Footprint" "Library:tcrt5000" (id 2) (at 231.14 69.342 0)
       (effects (font (size 1.27 1.27)) (justify left bottom) hide)
     )
@@
     (property "Reference" "U7" (id 0) (at 231.902 107.696 0))
     (property "Value" "TCRT5000" (id 1) (at 231.902 109.728 0))
-    (property "Footprint" "" (id 2) (at 231.902 115.824 0)
+    (property "Footprint" "Library:tcrt5000" (id 2) (at 231.902 115.824 0)
       (effects (font (size 1.27 1.27)) (justify left bottom) hide)
     )
@@
   (symbol (lib_id "Device:R_Small_US") (at 245.11 113.284 90) (unit 1)
     (in_bom yes) (on_board yes)
-    (property "Reference" "R7" (id 0) (at 245.11 115.316 90))
+    (property "Reference" "R9" (id 0) (at 245.11 115.316 90))
     (property "Value" "10kΩ" (id 1) (at 245.11 116.84 90))
     (property "Footprint" "Resistor_SMD:R_0805_2012Metric_Pad1.20x1.40mm_HandSolder" (id 2) (at 245.11 113.284 0)
@@
   (symbol (lib_id "Connector:Conn_01x04_Male") (at 198.12 113.538 0) (unit 1)
     (in_bom yes) (on_board yes)
-    (property "Reference" "J10" (id 0) (at 200.914 106.68 0))
+    (property "Reference" "J12" (id 0) (at 200.914 106.68 0))
     (property "Value" "Conn_01x04_Male" (id 1) (at 200.914 108.458 0))
-    (property "Footprint" "" (id 2) (at 198.12 113.538 0)
-      (effects (font (size 1.27 1.27)) hide)
-    )
+    (property "Footprint" "Connector_PinHeader_2.54mm:PinHeader_1x04_P2.54mm_Vertical" (id 2) (at 198.12 113.538 0)
+      (effects (font (size 1.27 1.27)) hide)
+    )

Commit message: 1.7
Connections:
- net A0: no longer J11.4 (Pin_4), J12.4 (Pin_4), J13.4 (Pin_4), R10.1, R8.1, R9.1, U6.COLL, U7.COLL, U8.COLL
- new net A1: J11.4 (Pin_4), R8.1, U6.COLL
- new net A2: J12.4 (Pin_4), R9.1, U7.COLL
- new net A3: J13.4 (Pin_4), R10.1, U8.COLL
Changed lines of the file:
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@@
     (stroke (width 0) (type default) (color 0 0 0 0))
   )
-  (label "A0" (at 241.3 110.744 0)
+  (label "A2" (at 203.2 118.618 0)
     (effects (font (size 1.27 1.27)) (justify left bottom))
   )
-  (label "A0" (at 240.792 87.376 0)
+  (label "A3" (at 241.554 133.858 0)
     (effects (font (size 1.27 1.27)) (justify left bottom))
   )
-  (label "A0" (at 203.2 118.618 0)
+  (label "A3" (at 203.454 141.732 0)
     (effects (font (size 1.27 1.27)) (justify left bottom))
   )
   (label "P5" (at 202.692 92.71 0)
+    (effects (font (size 1.27 1.27)) (justify left bottom))
+  )
+  (label "A1" (at 202.692 95.25 0)
     (effects (font (size 1.27 1.27)) (justify left bottom))
   )
@@
     (effects (font (size 1.27 1.27)) (justify left bottom))
   )
-  (label "A0" (at 241.554 133.858 0)
-    (effects (font (size 1.27 1.27)) (justify left bottom))
-  )
-  (label "A0" (at 202.692 95.25 0)
+  (label "A1" (at 240.792 87.376 0)
     (effects (font (size 1.27 1.27)) (justify left bottom))
   )
@@
     (effects (font (size 1.27 1.27)) (justify left bottom))
   )
+  (label "A2" (at 241.3 110.744 0)
+    (effects (font (size 1.27 1.27)) (justify left bottom))
+  )
   (label "GND" (at 202.438 67.056 0)
     (effects (font (size 1.27 1.27)) (justify left bottom))
@@
     (effects (font (size 1.27 1.27)) (justify left bottom))
   )
-  (label "A0" (at 203.454 141.732 0)
-    (effects (font (size 1.27 1.27)) (justify left bottom))
-  )

Commit message: 1.9
Parts:
- U5, U6, U7, U8: footprint Library:tcrt5000 -> Sumo:OPTO_TCRT5000
Changed lines of the file:
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@@
     (property "Reference" "U8" (id 0) (at 232.156 130.81 0))
     (property "Value" "TCRT5000" (id 1) (at 232.156 132.842 0))
-    (property "Footprint" "Library:tcrt5000" (id 2) (at 232.156 138.938 0)
+    (property "Footprint" "Sumo:OPTO_TCRT5000" (id 2) (at 232.156 138.938 0)
       (effects (font (size 1.27 1.27)) (justify left bottom) hide)
     )
@@
     (property "Reference" "U6" (id 0) (at 231.394 84.328 0))
     (property "Value" "TCRT5000" (id 1) (at 231.394 86.36 0))
-    (property "Footprint" "Library:tcrt5000" (id 2) (at 231.394 92.456 0)
+    (property "Footprint" "Sumo:OPTO_TCRT5000" (id 2) (at 231.394 92.456 0)
       (effects (font (size 1.27 1.27)) (justify left bottom) hide)
     )
@@
     (property "Reference" "U5" (id 0) (at 231.14 61.214 0))
     (property "Value" "TCRT5000" (id 1) (at 231.14 63.246 0))
-    (property "Footprint" "Library:tcrt5000" (id 2) (at 231.14 69.342 0)
+    (property "Footprint" "Sumo:OPTO_TCRT5000" (id 2) (at 231.14 69.342 0)
       (effects (font (size 1.27 1.27)) (justify left bottom) hide)
     )
@@
     (property "Reference" "U7" (id 0) (at 231.902 107.696 0))
     (property "Value" "TCRT5000" (id 1) (at 231.902 109.728 0))
-    (property "Footprint" "Library:tcrt5000" (id 2) (at 231.902 115.824 0)
-      (effects (font (size 1.27 1.27)) (justify left bottom) hide)
-    )
+    (property "Footprint" "Sumo:OPTO_TCRT5000" (id 2) (at 231.902 115.824 0)
+      (effects (font (size 1.27 1.27)) (justify left bottom) hide)
+    )

Commit message: 2.0 alabama
Parts:
- removed J7, J8: IR204, LED_THT:LED_D1.8mm_W1.8mm_H2.4mm_Horizontal_O6.35mm_Z8.2mm, symbol Connector:Conn_01x02_Male
- added C?: 100uf, symbol Device:C_Small
- added R?: 100Ω, symbol Device:R_Small_US
- added R?: 20kΩ, symbol Device:R_Small_US
- J9: footprint Package_TO_SOT_THT:TO-92L_Inline_Wide -> Connector_PinHeader_2.54mm:PinHeader_1x03_P2.54mm_Vertical
Connections:
- net at J9.1 (Pin_1): now also R?.1
- new net 3.3V: R?.2
Other:
- moved on the sheet: J9
Changed lines of the file:
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@@
   (junction (at 240.538 66.802) (diameter 0) (color 0 0 0 0)
   )
+  (junction (at 173.99 99.822) (diameter 0) (color 0 0 0 0)
+  )
   (junction (at 241.3 113.284) (diameter 0) (color 0 0 0 0)
   )
@@
     (stroke (width 0) (type default) (color 0 0 0 0))
   )
+  (wire (pts (xy 170.942 99.822) (xy 173.99 99.822))
+    (stroke (width 0) (type default) (color 0 0 0 0))
+  )
   (wire (pts (xy 224.282 123.698) (xy 232.156 123.698))
     (stroke (width 0) (type default) (color 0 0 0 0))
@@
     (stroke (width 0) (type default) (color 0 0 0 0))
   )
+  (wire (pts (xy 173.99 95.504) (xy 173.99 99.822))
+    (stroke (width 0) (type default) (color 0 0 0 0))
+  )
   (wire (pts (xy 240.538 64.262) (xy 240.538 66.802))
     (stroke (width 0) (type default) (color 0 0 0 0))
@@
     (stroke (width 0) (type default) (color 0 0 0 0))
   )
+  (wire (pts (xy 165.862 99.822) (xy 161.798 99.822))
+    (stroke (width 0) (type default) (color 0 0 0 0))
+  )
   (wire (pts (xy 232.156 123.698) (xy 232.156 124.46))
     (stroke (width 0) (type default) (color 0 0 0 0))
@@
     (stroke (width 0) (type default) (color 0 0 0 0))
   )
+  (wire (pts (xy 161.798 99.822) (xy 161.798 97.536))
+    (stroke (width 0) (type default) (color 0 0 0 0))
+  )
   (wire (pts (xy 231.648 100.33) (xy 239.014 100.33))
     (stroke (width 0) (type default) (color 0 0 0 0))
@@
     (stroke (width 0) (type default) (color 0 0 0 0))
   )
+  (wire (pts (xy 173.99 99.822) (xy 173.99 113.538))
+    (stroke (width 0) (type default) (color 0 0 0 0))
+  )
   (wire (pts (xy 214.63 92.71) (xy 214.63 89.916))
     (stroke (width 0) (type default) (color 0 0 0 0))
@@
     (effects (font (size 1.27 1.27)) (justify left bottom))
   )
+  (label "3.3V" (at 173.99 95.504 0)
+    (effects (font (size 1.27 1.27)) (justify left bottom))
+  )
   (label "A0" (at 202.438 72.136 0)
     (effects (font (size 1.27 1.27)) (justify left bottom))
@@
   (label "5V" (at 247.904 136.398 0)
     (effects (font (size 1.27 1.27)) (justify left bottom))
+  )
+  (symbol (lib_id "Device:R_Small_US") (at 168.402 99.822 90) (unit 1)
+    (in_bom yes) (on_board yes)
+    (property "Reference" "R?" (id 0) (at 168.402 96.012 90))
+    (property "Value" "100Ω" (id 1) (at 168.402 97.79 90))
+    (property "Footprint" "" (id 2) (at 168.402 99.822 0)
+      (effects (font (size 1.27 1.27)) hide)
+    )
+    (property "Datasheet" "~" (id 3) (at 168.402 99.822 0)
+      (effects (font (size 1.27 1.27)) hide)
+    )
+    (pin "1")
+    (pin "2")
   )
   (symbol (lib_id "Device:R_Small_US") (at 244.348 66.802 90) (unit 1)
@@
     (pin "2")
   )
+  (symbol (lib_id "Device:C_Small") (at 168.656 112.268 90) (unit 1)
+    (in_bom yes) (on_board yes)
+    (property "Reference" "C?" (id 0) (at 168.656 108.204 90))
+    (property "Value" "100uf" (id 1) (at 168.656 109.728 90))
+    (property "Footprint" "" (id 2) (at 168.656 112.268 0)
+      (effects (font (size 1.27 1.27)) hide)
+    )
+    (property "Datasheet" "~" (id 3) (at 168.656 112.268 0)
+      (effects (font (size 1.27 1.27)) hide)
+    )
+    (pin "1")
+    (pin "2")
+  )
   (symbol (lib_id "power:GND") (at 231.648 101.092 0) (unit 1)
     (in_bom yes) (on_board yes) (fields_autoplaced)
@@
     (pin "1")
   )
-  (symbol (lib_id "Connector:Conn_01x03_Male") (at 108.712 105.156 180) (unit 1)
-    (in_bom yes) (on_board yes)
-    (property "Reference" "J9" (id 0) (at 109.982 103.886 0)
+  (symbol (lib_id "Connector:Conn_01x03_Male") (at 159.258 92.456 270) (unit 1)
+    (in_bom yes) (on_board yes)
+    (property "Reference" "J9" (id 0) (at 160.274 89.662 90)
       (effects (font (size 1.27 1.27)) (justify right))
     )
-    (property "Value" "TL1838" (id 1) (at 109.22 106.426 0)
+    (property "Value" "TL1838" (id 1) (at 162.814 91.44 90)
       (effects (font (size 1.27 1.27)) (justify right))
     )
-    (property "Footprint" "Package_TO_SOT_THT:TO-92L_Inline_Wide" (id 2) (at 108.712 105.156 0)
-      (effects (font (size 1.27 1.27)) hide)
-    )
-    (property "Datasheet" "~" (id 3) (at 108.712 105.156 0)
+    (property "Footprint" "Connector_PinHeader_2.54mm:PinHeader_1x03_P2.54mm_Vertical" (id 2) (at 159.258 92.456 0)
+      (effects (font (size 1.27 1.27)) hide)
+    )
+    (property "Datasheet" "~" (id 3) (at 159.258 92.456 0)
       (effects (font (size 1.27 1.27)) hide)
     )
@@
     )
     (property "Datasheet" "~" (id 3) (at 245.364 136.398 0)
-      (effects (font (size 1.27 1.27)) hide)
-    )
-    (pin "1")
-    (pin "2")
-  )
-  (symbol (lib_id "Connector:Conn_01x02_Male") (at 108.712 97.79 180) (unit 1)
-    (in_bom yes) (on_board yes) (fields_autoplaced)
-    (property "Reference" "J8" (id 0) (at 110.236 95.2499 0)
-      (effects (font (size 1.27 1.27)) (justify right))
-    )
-    (property "Value" "IR204" (id 1) (at 110.236 97.7899 0)
-      (effects (font (size 1.27 1.27)) (justify right))
-    )
-    (property "Footprint" "LED_THT:LED_D1.8mm_W1.8mm_H2.4mm_Horizontal_O6.35mm_Z8.2mm" (id 2) (at 108.712 97.79 0)
-      (effects (font (size 1.27 1.27)) hide)
-    )
-    (property "Datasheet" "~" (id 3) (at 108.712 97.79 0)
       (effects (font (size 1.27 1.27)) hide)
     )
@@
     (pin "4")
   )
-  (symbol (lib_id "Connector:Conn_01x02_Male") (at 108.712 90.424 180) (unit 1)
-    (in_bom yes) (on_board yes) (fields_autoplaced)
-    (property "Reference" "J7" (id 0) (at 110.236 87.8839 0)
-      (effects (font (size 1.27 1.27)) (justify right))
-    )
-    (property "Value" "IR204" (id 1) (at 110.236 90.4239 0)
-      (effects (font (size 1.27 1.27)) (justify right))
-    )
-    (property "Footprint" "LED_THT:LED_D1.8mm_W1.8mm_H2.4mm_Horizontal_O6.35mm_Z8.2mm" (id 2) (at 108.712 90.424 0)
-      (effects (font (size 1.27 1.27)) hide)
-    )
-    (property "Datasheet" "~" (id 3) (at 108.712 90.424 0)
-      (effects (font (size 1.27 1.27)) hide)
-    )
-    (pin "1")
-    (pin "2")
-  )
   (symbol (lib_id "Device:R_Small_US") (at 244.602 89.916 90) (unit 1)
     (in_bom yes) (on_board yes)
@@
       (effects (font (size 1.27 1.27)) hide)
     )
+    (pin "1")
+    (pin "2")
+  )
+  (symbol (lib_id "Device:R_Small_US") (at 168.402 106.172 90) (unit 1)
+    (in_bom yes) (on_board yes)
+    (property "Reference" "R?" (id 0) (at 168.402 102.362 90))
+    (property "Value" "20kΩ" (id 1) (at 168.402 104.14 90))
+    (property "Footprint" "" (id 2) (at 168.402 106.172 0)
+      (effects (font (size 1.27 1.27)) hide)
+    )
+    (property "Datasheet" "~" (id 3) (at 168.402 106.172 0)
+      (effects (font (size 1.27 1.27)) hide)
+    )

Commit message: 2.1 Missouri
Parts:
- removed J10, J11, J12, J13: Conn_01x04_Male, Connector_PinHeader_2.54mm:PinHeader_1x04_P2.54mm_Vertical, symbol Connector:Conn_01x04_Male
- removed R10, R7, R8, R9: 10kΩ, Resistor_SMD:R_0805_2012Metric_Pad1.20x1.40mm_HandSolder, symbol Device:R_Small_US
- added J10, J11, J7, J8: Conn_01x03_Male, Connector_PinHeader_2.54mm:PinHeader_1x03_P2.54mm_Vertical, symbol Connector:Conn_01x03_Male
- added RV1, RV2, RV3, RV4: 100k, Potentiometer_THT:Potentiometer_ACP_CA6-H2,5_Horizontal, symbol Device:R_Potentiometer_US
- C13: renamed from C?; footprint (none) -> Capacitor_SMD:C_0805_2012Metric_Pad1.18x1.45mm_HandSolder
- R7, R8: renamed from R?; footprint (none) -> Resistor_SMD:R_0805_2012Metric_Pad1.20x1.40mm_HandSolder
Connections:
- net P4 is gone; now on net 3.3V: R3.1
- net P5 is gone; now on net 3.3V: R4.1
- net P6 is gone; now on net 3.3V: R5.1
- net P7 is gone; now on net 3.3V: R6.1
- net 3.3V: now also J10.1 (Pin_1), J11.1 (Pin_1), J7.1 (Pin_1), J8.1 (Pin_1), RV1.1, RV1.2, RV2.1, RV2.2, RV3.1, RV3.2, RV4.1, RV4.2; no longer R7.2
- net A0: now also J7.3 (Pin_3), RV1.3
- net A1: now also J8.3 (Pin_3), RV2.3
- net A2: now also J10.3 (Pin_3), RV3.3
- net A3: now also J11.3 (Pin_3), RV4.3
- net GND: now also C13.1, J9.2 (Pin_2), J10.2 (Pin_2), J11.2 (Pin_2), J7.2 (Pin_2), J8.2 (Pin_2)
- net at C13.2: now also R7.2, R8.2
- net at J9.3 (Pin_3): now also R8.1
Other:
- moved on the sheet: C13, J9, R7, R8
