File: PCB/Carte Mere/Capteur infrarouge.kicad_sch (KiCad schematic)
At the start: 20 parts, among them J10 Conn_01x03_Male, J11 Conn_01x03_Male, J7 Conn_01x03_Male, J8 Conn_01x03_Male, J9 TL1838, U5 TCRT5000, U6 TCRT5000, U7 TCRT5000, U8 TCRT5000

Commit message: 2.2 Florida
Connections:
- net 3.3V: now also C13.2, R7.2, R8.2
- net P8: now reaches J9.3 (Pin_3), R8.1
Other:
- moved on the sheet: C13, J9, R7, R8
Changed lines of the file:
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@@
   (junction (at 240.538 66.802) (diameter 0) (color 0 0 0 0)
   )
-  (junction (at 154.94 95.504) (diameter 0) (color 0 0 0 0)
-  )
-  (junction (at 140.208 95.504) (diameter 0) (color 0 0 0 0)
-  )
-  (junction (at 154.94 89.408) (diameter 0) (color 0 0 0 0)
+  (junction (at 182.88 100.838) (diameter 0) (color 0 0 0 0)
+  )
+  (junction (at 168.148 100.838) (diameter 0) (color 0 0 0 0)
+  )
+  (junction (at 182.88 94.742) (diameter 0) (color 0 0 0 0)
   )
   (junction (at 241.3 113.284) (diameter 0) (color 0 0 0 0)
@@
     (stroke (width 0) (type default) (color 0 0 0 0))
   )
-  (wire (pts (xy 151.892 89.408) (xy 154.94 89.408))
+  (wire (pts (xy 179.832 94.742) (xy 182.88 94.742))
     (stroke (width 0) (type default) (color 0 0 0 0))
   )
@@
     (stroke (width 0) (type default) (color 0 0 0 0))
   )
-  (wire (pts (xy 154.94 102.362) (xy 152.146 102.362))
+  (wire (pts (xy 182.88 107.696) (xy 180.086 107.696))
     (stroke (width 0) (type default) (color 0 0 0 0))
   )
@@
     (stroke (width 0) (type default) (color 0 0 0 0))
   )
-  (wire (pts (xy 154.94 85.09) (xy 154.94 89.408))
-    (stroke (width 0) (type default) (color 0 0 0 0))
-  )
-  (wire (pts (xy 140.208 95.504) (xy 140.208 87.122))
+  (wire (pts (xy 182.88 90.424) (xy 182.88 94.742))
+    (stroke (width 0) (type default) (color 0 0 0 0))
+  )
+  (wire (pts (xy 168.148 100.838) (xy 168.148 92.456))
     (stroke (width 0) (type default) (color 0 0 0 0))
   )
@@
     (stroke (width 0) (type default) (color 0 0 0 0))
   )
-  (wire (pts (xy 154.94 95.504) (xy 154.94 102.362))
+  (wire (pts (xy 182.88 100.838) (xy 182.88 107.696))
     (stroke (width 0) (type default) (color 0 0 0 0))
   )
@@
     (stroke (width 0) (type default) (color 0 0 0 0))
   )
-  (wire (pts (xy 146.812 89.408) (xy 142.748 89.408))
+  (wire (pts (xy 174.752 94.742) (xy 170.688 94.742))
     (stroke (width 0) (type default) (color 0 0 0 0))
   )
@@
     (stroke (width 0) (type default) (color 0 0 0 0))
   )
-  (wire (pts (xy 142.748 89.408) (xy 142.748 87.122))
+  (wire (pts (xy 170.688 94.742) (xy 170.688 92.456))
     (stroke (width 0) (type default) (color 0 0 0 0))
   )
@@
     (stroke (width 0) (type default) (color 0 0 0 0))
   )
-  (wire (pts (xy 137.668 102.362) (xy 137.668 87.122))
+  (wire (pts (xy 165.608 107.696) (xy 165.608 92.456))
     (stroke (width 0) (type default) (color 0 0 0 0))
   )
@@
     (stroke (width 0) (type default) (color 0 0 0 0))
   )
-  (wire (pts (xy 146.812 95.504) (xy 140.208 95.504))
+  (wire (pts (xy 174.752 100.838) (xy 168.148 100.838))
     (stroke (width 0) (type default) (color 0 0 0 0))
   )
@@
     (stroke (width 0) (type default) (color 0 0 0 0))
   )
-  (wire (pts (xy 151.892 95.504) (xy 154.94 95.504))
+  (wire (pts (xy 179.832 100.838) (xy 182.88 100.838))
     (stroke (width 0) (type default) (color 0 0 0 0))
   )
@@
     (stroke (width 0) (type default) (color 0 0 0 0))
   )
-  (wire (pts (xy 154.94 89.408) (xy 154.94 95.504))
+  (wire (pts (xy 182.88 94.742) (xy 182.88 100.838))
     (stroke (width 0) (type default) (color 0 0 0 0))
   )
@@
     (stroke (width 0) (type default) (color 0 0 0 0))
   )
-  (wire (pts (xy 147.066 102.362) (xy 137.668 102.362))
+  (wire (pts (xy 175.006 107.696) (xy 165.608 107.696))
     (stroke (width 0) (type default) (color 0 0 0 0))
   )
@@
     (effects (font (size 1.27 1.27)) (justify left bottom))
   )
-  (symbol (lib_id "Device:R_Small_US") (at 149.352 89.408 90) (unit 1)
-    (in_bom yes) (on_board yes)
-    (property "Reference" "R7" (id 0) (at 149.352 85.598 90))
-    (property "Value" "100Ω" (id 1) (at 149.352 87.376 90))
-    (property "Footprint" "Resistor_SMD:R_0805_2012Metric_Pad1.20x1.40mm_HandSolder" (id 2) (at 149.352 89.408 0)
-      (effects (font (size 1.27 1.27)) hide)
-    )
-    (property "Datasheet" "~" (id 3) (at 149.352 89.408 0)
-      (effects (font (size 1.27 1.27)) hide)
-    )
-    (pin "1")
-    (pin "2")
-  )
-  (symbol (lib_id "Device:C_Small") (at 149.352 95.504 90) (unit 1)
-    (in_bom yes) (on_board yes)
-    (property "Reference" "C13" (id 0) (at 149.352 91.44 90))
-    (property "Value" "100uf" (id 1) (at 149.352 92.964 90))
-    (property "Footprint" "Capacitor_SMD:C_0805_2012Metric_Pad1.18x1.45mm_HandSolder" (id 2) (at 149.352 95.504 0)
-      (effects (font (size 1.27 1.27)) hide)
-    )
-    (property "Datasheet" "~" (id 3) (at 149.352 95.504 0)
+  (global_label "P8" (shape input) (at 165.608 107.696 180) (fields_autoplaced)
+    (effects (font (size 1.27 1.27)) (justify right))
+    (property "Intersheet References" "${INTERSHEET_REFS}" (id 0) (at 160.7154 107.6166 0)
+      (effects (font (size 1.27 1.27)) (justify right) hide)
+    )
+  )
+  (global_label "3.3V" (shape input) (at 182.88 90.424 0) (fields_autoplaced)
+    (effects (font (size 1.27 1.27)) (justify left))
+    (property "Intersheet References" "${INTERSHEET_REFS}" (id 0) (at 189.4055 90.3446 0)
+      (effects (font (size 1.27 1.27)) (justify left) hide)
+    )
+  )
+  (symbol (lib_id "Device:R_Small_US") (at 177.292 94.742 90) (unit 1)
+    (in_bom yes) (on_board yes)
+    (property "Reference" "R7" (id 0) (at 177.292 90.932 90))
+    (property "Value" "100Ω" (id 1) (at 177.292 92.71 90))
+    (property "Footprint" "Resistor_SMD:R_0805_2012Metric_Pad1.20x1.40mm_HandSolder" (id 2) (at 177.292 94.742 0)
+      (effects (font (size 1.27 1.27)) hide)
+    )
+    (property "Datasheet" "~" (id 3) (at 177.292 94.742 0)
+      (effects (font (size 1.27 1.27)) hide)
+    )
+    (pin "1")
+    (pin "2")
+  )
+  (symbol (lib_id "Device:C_Small") (at 177.292 100.838 90) (unit 1)
+    (in_bom yes) (on_board yes)
+    (property "Reference" "C13" (id 0) (at 177.292 96.774 90))
+    (property "Value" "100uf" (id 1) (at 177.292 98.298 90))
+    (property "Footprint" "Capacitor_SMD:C_0805_2012Metric_Pad1.18x1.45mm_HandSolder" (id 2) (at 177.292 100.838 0)
+      (effects (font (size 1.27 1.27)) hide)
+    )
+    (property "Datasheet" "~" (id 3) (at 177.292 100.838 0)
       (effects (font (size 1.27 1.27)) hide)
     )
@@
     (pin "1")
   )
-  (symbol (lib_id "Connector:Conn_01x03_Male") (at 140.208 82.042 270) (unit 1)
-    (in_bom yes) (on_board yes)
-    (property "Reference" "J9" (id 0) (at 141.224 79.248 90)
+  (symbol (lib_id "Connector:Conn_01x03_Male") (at 168.148 87.376 270) (unit 1)
+    (in_bom yes) (on_board yes)
+    (property "Reference" "J9" (id 0) (at 169.164 84.582 90)
       (effects (font (size 1.27 1.27)) (justify right))
     )
-    (property "Value" "TL1838" (id 1) (at 143.764 81.026 90)
+    (property "Value" "TL1838" (id 1) (at 171.704 86.36 90)
       (effects (font (size 1.27 1.27)) (justify right))
     )
-    (property "Footprint" "Connector_PinHeader_2.54mm:PinHeader_1x03_P2.54mm_Vertical" (id 2) (at 140.208 82.042 0)
-      (effects (font (size 1.27 1.27)) hide)
-    )
-    (property "Datasheet" "~" (id 3) (at 140.208 82.042 0)
+    (property "Footprint" "Connector_PinHeader_2.54mm:PinHeader_1x03_P2.54mm_Vertical" (id 2) (at 168.148 87.376 0)
+      (effects (font (size 1.27 1.27)) hide)
+    )
+    (property "Datasheet" "~" (id 3) (at 168.148 87.376 0)
       (effects (font (size 1.27 1.27)) hide)
     )
@@
     (pin "E")
   )
-  (symbol (lib_id "power:GND") (at 140.208 95.504 0) (unit 1)
-    (in_bom yes) (on_board yes)
-    (property "Reference" "#PWR0101" (id 0) (at 140.208 101.854 0)
-      (effects (font (size 1.27 1.27)) hide)
-    )
-    (property "Value" "GND" (id 1) (at 140.208 99.06 0))
-    (property "Footprint" "" (id 2) (at 140.208 95.504 0)
-      (effects (font (size 1.27 1.27)) hide)
-    )
-    (property "Datasheet" "" (id 3) (at 140.208 95.504 0)
-      (effects (font (size 1.27 1.27)) hide)
-    )
-    (pin "1")
-  )
-  (symbol (lib_id "Device:R_Small_US") (at 149.606 102.362 90) (unit 1)
-    (in_bom yes) (on_board yes)
-    (property "Reference" "R8" (id 0) (at 149.606 98.552 90))
-    (property "Value" "20kΩ" (id 1) (at 149.606 100.33 90))
-    (property "Footprint" "Resistor_SMD:R_0805_2012Metric_Pad1.20x1.40mm_HandSolder" (id 2) (at 149.606 102.362 0)
-      (effects (font (size 1.27 1.27)) hide)
-    )
-    (property "Datasheet" "~" (id 3) (at 149.606 102.362 0)
-      (effects (font (size 1.27 1.27)) hide)
-    )
+  (symbol (lib_id "power:GND") (at 168.148 100.838 0) (unit 1)
+    (in_bom yes) (on_board yes)
+    (property "Reference" "#PWR0101" (id 0) (at 168.148 107.188 0)
+      (effects (font (size 1.27 1.27)) hide)
+    )
+    (property "Value" "GND" (id 1) (at 168.148 104.394 0))
+    (property "Footprint" "" (id 2) (at 168.148 100.838 0)
+      (effects (font (size 1.27 1.27)) hide)
+    )
+    (property "Datasheet" "" (id 3) (at 168.148 100.838 0)
+      (effects (font (size 1.27 1.27)) hide)
+    )
+    (pin "1")
+  )
+  (symbol (lib_id "Device:R_Small_US") (at 177.546 107.696 90) (unit 1)
+    (in_bom yes) (on_board yes)
+    (property "Reference" "R8" (id 0) (at 177.546 103.886 90))
+    (property "Value" "20kΩ" (id 1) (at 177.546 105.664 90))
+    (property "Footprint" "Resistor_SMD:R_0805_2012Metric_Pad1.20x1.40mm_HandSolder" (id 2) (at 177.546 107.696 0)
+      (effects (font (size 1.27 1.27)) hide)
+    )
+    (property "Datasheet" "~" (id 3) (at 177.546 107.696 0)
+      (effects (font (size 1.27 1.27)) hide)
+    )
