File: PCB/Carte Mere/untitled.kicad_sch (KiCad schematic)
At the start: 18 parts

Commit message: lol
Parts:
- removed C? (x4): 0.1uf, symbol Device:C
- removed D? (x4): D, symbol Device:D
- removed R? (x2): R_US, symbol Device:R_US
- removed U? (x2): ZXBM5210-S, Package_SO:SOIC-8_3.9x4.9mm_P1.27mm, symbol Driver_Motor:ZXBM5210-S
- removed U?: LM1117-3.3, symbol Regulator_Linear:LM1117-3.3
- added C1, C2, C5, C6: 0.47uf, symbol Device:C
- added C3, C4, C7, C8: 0.1uf, symbol Device:C
- added D1, D3: Verte, Diode_SMD:D_0805_2012Metric_Pad1.15x1.40mm_HandSolder, symbol Device:LED
- added D2, D4: Rouge, Diode_SMD:D_0805_2012Metric_Pad1.15x1.40mm_HandSolder, symbol Device:LED
- added J1, J2: 01x20_Female, symbol Connector:Conn_01x20_Female
- added J3, J4: 01x02_Male, symbol Connector:Conn_01x02_Male
- added J?: TL1838, symbol Connector:Conn_01x03_Male
- added J? (x4): TRCT5000, symbol Connector_Generic:Conn_02x02_Counter_Clockwise
- added J? (x2): IR204, symbol Connector:Conn_01x02_Male
- added JP1: Jumper_3_Bridge, symbol Jumper:Jumper_3_Bridged12
- added R1, R2: 330, symbol Device:R_US
- added R? (x4): 500Ω, symbol Device:R_Small_US
- added R? (x4): 10kΩ, symbol Device:R_Small_US
- added U1, U2: ZXBM5210-S, Package_SO:SOIC-8_3.9x4.9mm_P1.27mm, symbol Driver_Motor:ZXBM5210-S
- added U?: LD1117S33TR_SOT223, Package_TO_SOT_SMD:SOT-223-3_TabPin2, symbol Regulator_Linear:LD1117S33TR_SOT223
- C11: renamed from C?; value 10uf -> 100nf
- gave numbers to parts that had none: 4
Connections:
- net 5V: now also J1.11 (Pin_11), JP1.1 (A)
- net GND: now also C1.2, C2.2, C3.2, C4.2, C5.2, C6.2, C7.2, C8.2, J1.10 (Pin_10), J1.12 (Pin_12), J2.9 (Pin_9), J?.3 (Pin_3), J?.3 (Pin_3), J?.3 (Pin_3), J?.3 (Pin_3), J?.4 (Pin_4), J?.4 (Pin_4), J?.4 (Pin_4), J?.4 (Pin_4), U1.8 (GND), U2.8 (GND), U?.1 (GND)
- net 9V: now reaches C9.1, U3.4 (VIN)
- net 9V: now also JP1.3 (B)
- net at C11.1: now also JP1.2 (C), U?.3 (VI)
- net 3.3V: now reaches C12.1
- net 3.3V: now also J1.9 (Pin_9), J2.10 (Pin_10), U?.2 (VO)
- new net: R1.1, U1.5 (REV)
- new net: D1.1 (K), D2.2 (A), R1.2
- new net: D1.2 (A), D2.1 (K), U1.4 (FWD)
- new net: C7.1, J4.2 (Pin_2), U2.7 (OUT2)
- new net: J?.1 (Pin_1), R?.2 (x4)
- new net: C8.1, J4.1 (Pin_1), U2.1 (OUT1)
- new net: R2.1, U2.5 (REV)
- new net: D3.1 (K), D4.2 (A), R2.2
- new net: J?.2 (Pin_2), R?.2 (x4)
- new net: C4.1, J3.1 (Pin_1), U1.1 (OUT1)
- new net: D3.2 (A), D4.1 (K), U2.4 (FWD)
- new net: C3.1, J3.2 (Pin_2), U1.7 (OUT2)
- new net 6V: C1.1, C2.1, C5.1, C6.1, U1.2 (VM), U1.3 (VDD), U1.6 (VREF), U2.2 (VM), U2.3 (VDD), U2.6 (VREF)
- new net P0: J2.1 (Pin_1)
- new net P1: J2.2 (Pin_2)
- new net P10: J2.15 (Pin_15)
- new net P11: J2.16 (Pin_16)
- new net P12: J2.17 (Pin_17)
- new net P13: J2.18 (Pin_18)
- new net P14: J2.19 (Pin_19)
- new net P15: J2.20 (Pin_20)
- new net P16: J1.20 (Pin_20)
- new net P17: J1.19 (Pin_19)
- new net P18: J1.18 (Pin_18)
- new net P19: J1.17 (Pin_17)
- new net P2: J2.3 (Pin_3)
- new net P20: J1.16 (Pin_16)
- new net P21: J1.15 (Pin_15)
- new net P22: J1.14 (Pin_14)
- new net P23: J1.13 (Pin_13)
- new net P24: J1.8 (Pin_8)
- new net P25: J1.7 (Pin_7)
- new net P26: J1.6 (Pin_6)
- new net P27: J1.5 (Pin_5)
- new net P28_SCL: J1.4 (Pin_4)
- new net P29_SDA: J1.3 (Pin_3)
- new net P3: J2.4 (Pin_4)
- new net P30_TX: J1.2 (Pin_2)
- new net P31_RX: J1.1 (Pin_1)
- new net P4: J2.5 (Pin_5)
- new net P5: J2.6 (Pin_6)
- new net P6: J2.7 (Pin_7)
- new net P7: J2.8 (Pin_8)
- new net P8: J2.13 (Pin_13)
- new net P9: J2.14 (Pin_14)
- new net RESET: J2.11 (Pin_11)
Other:
- moved on the sheet: C10, C11, C12, C9, U3

Commit message: Version 1.0
Parts:
- removed C3, C4, C7, C8: 0.1uf, symbol Device:C
- removed C5, C6: 0.47uf, symbol Device:C
- removed D3: Verte, Diode_SMD:D_0805_2012Metric_Pad1.15x1.40mm_HandSolder, symbol Device:LED
- removed D4: Rouge, Diode_SMD:D_0805_2012Metric_Pad1.15x1.40mm_HandSolder, symbol Device:LED
- removed J4: 01x02_Male, symbol Connector:Conn_01x02_Male
- removed R2: 330, symbol Device:R_US
- removed U2: ZXBM5210-S, Package_SO:SOIC-8_3.9x4.9mm_P1.27mm, symbol Driver_Motor:ZXBM5210-S
- added C? (x4): 0.1uf, symbol Device:C
- added C? (x2): 0.47uf, symbol Device:C
- added D?: Verte, Diode_SMD:D_0805_2012Metric_Pad1.15x1.40mm_HandSolder, symbol Device:LED
- added D?: Rouge, Diode_SMD:D_0805_2012Metric_Pad1.15x1.40mm_HandSolder, symbol Device:LED
- added J?: Moteur, symbol Connector:Conn_01x02_Male
- added R?: 330, symbol Device:R_US
- added U?: ZXBM5210-S, Package_SO:SOIC-8_3.9x4.9mm_P1.27mm, symbol Driver_Motor:ZXBM5210-S
- J3: value 01x02_Male -> Moteur
Connections:
- net 6V: now also C?.1, C?.1, U?.2 (VM), U?.3 (VDD), U?.6 (VREF)
- net GND: now also C?.2, C?.2, C?.2, C?.2, C?.2, C?.2, U?.8 (GND)
- net at R1.1: now also J3.1 (Pin_1), U1.7 (OUT2), C?.1; no longer U1.5 (REV)
- net at D1.2 (A), D2.1 (K): now also J3.2 (Pin_2), U1.1 (OUT1), C?.1; no longer U1.4 (FWD)
- new net: C?.1, J?.1 (Pin_1), R?.1, U?.7 (OUT2)
- new net: C?.1, D?.1 (K), D?.2 (A), J?.2 (Pin_2), U?.1 (OUT1)
- new net: D?.1 (K), D?.2 (A), R?.2
Other:
- moved on the sheet: C1, C2, D1, D2, J3, R1, U1

Commit message: 1.2 PCB
Parts:
- removed J?: TL1838, symbol Connector:Conn_01x03_Male
- removed J? (x4): TRCT5000, symbol Connector_Generic:Conn_02x02_Counter_Clockwise
- removed J? (x2): IR204, symbol Connector:Conn_01x02_Male
- removed R? (x4): 500Ω, symbol Device:R_Small_US
- removed R? (x4): 10kΩ, symbol Device:R_Small_US
- added J12: Alim 6V, Connector_PinHeader_2.54mm:PinHeader_1x02_P2.54mm_Vertical, symbol Connector:Conn_01x02_Male
- added J13: Alim 9V, Connector_PinHeader_2.54mm:PinHeader_1x02_P2.54mm_Vertical, symbol Connector:Conn_01x02_Male
- C1, C2: value 0.47uf -> 1uf; footprint (none) -> Capacitor_SMD:C_0805_2012Metric_Pad1.18x1.45mm_HandSolder
- C10, C11, C3, C4: renamed from C?; footprint (none) -> Capacitor_SMD:C_0805_2012Metric_Pad1.18x1.45mm_HandSolder
- C6, C7: renamed from C?; value 0.47uf -> 1uf; footprint (none) -> Capacitor_SMD:C_0805_2012Metric_Pad1.18x1.45mm_HandSolder
- J1: renamed from J3; footprint (none) -> Connector_PinHeader_2.54mm:PinHeader_1x02_P2.54mm_Vertical
- J2: renamed from J?; footprint (none) -> Connector_PinHeader_2.54mm:PinHeader_1x02_P2.54mm_Vertical
- J3: renamed from J1; footprint (none) -> Connector_PinSocket_2.54mm:PinSocket_1x20_P2.54mm_Vertical
- J4: renamed from J2; footprint (none) -> Connector_PinSocket_2.54mm:PinSocket_1x20_P2.54mm_Vertical
- JP1: footprint (none) -> Connector_PinHeader_2.54mm:PinHeader_1x03_P2.54mm_Vertical
- R1: footprint (none) -> Resistor_SMD:R_0805_2012Metric_Pad1.20x1.40mm_HandSolder
- R2: renamed from R?; footprint (none) -> Resistor_SMD:R_0805_2012Metric_Pad1.20x1.40mm_HandSolder
- U4: renamed from U?; footprint Package_TO_SOT_SMD:SOT-223-3_TabPin2 -> Package_TO_SOT_SMD:TO-252-2
- gave numbers to parts that had none: 3
- renumbered C9 to C5, C10 to C8, C11 to C9, U3 to U2
Connections:
- net P0: now also U1.4 (FWD)
- net P1: now also U1.5 (REV)
- net P2: now also U3.4 (FWD)
- net P3: now also U3.5 (REV)

Commit message: 1.4 Carte mere
Connections:
- net 6V: now also J12.1 (Pin_1)
- net 9V: now also J13.1 (Pin_1)
- net GND: now also J12.2 (Pin_2), J13.2 (Pin_2)
Other:
- moved on the sheet: J12, J13
Changed lines of the file:
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@@
   (junction (at 158.496 56.388) (diameter 0) (color 0 0 0 0)
   )
+  (junction (at 110.744 56.388) (diameter 0) (color 0 0 0 0)
+  )
   (junction (at 99.822 101.6) (diameter 0) (color 0 0 0 0)
   )
@@
   (junction (at 166.116 101.6) (diameter 0) (color 0 0 0 0)
   )
+  (junction (at 110.744 43.688) (diameter 0) (color 0 0 0 0)
+  )
   (junction (at 152.908 111.506) (diameter 0) (color 0 0 0 0)
   )
@@
   (junction (at 152.908 119.126) (diameter 0) (color 0 0 0 0)
   )
+  (junction (at 64.008 106.426) (diameter 0) (color 0 0 0 0)
+  )
   (junction (at 86.614 111.506) (diameter 0) (color 0 0 0 0)
   )
@@
     (stroke (width 0) (type default) (color 0 0 0 0))
   )
+  (wire (pts (xy 45.72 96.266) (xy 53.848 96.266))
+    (stroke (width 0) (type default) (color 0 0 0 0))
+  )
   (wire (pts (xy 130.302 106.426) (xy 130.302 107.696))
     (stroke (width 0) (type default) (color 0 0 0 0))
@@
     (stroke (width 0) (type default) (color 0 0 0 0))
   )
+  (wire (pts (xy 102.616 43.688) (xy 110.744 43.688))
+    (stroke (width 0) (type default) (color 0 0 0 0))
+  )
   (wire (pts (xy 99.822 110.236) (xy 99.822 113.03))
     (stroke (width 0) (type default) (color 0 0 0 0))
@@
     (stroke (width 0) (type default) (color 0 0 0 0))
   )
+  (wire (pts (xy 45.72 98.806) (xy 45.72 106.426))
+    (stroke (width 0) (type default) (color 0 0 0 0))
+  )
   (wire (pts (xy 170.942 92.71) (xy 166.116 92.71))
     (stroke (width 0) (type default) (color 0 0 0 0))
@@
     (stroke (width 0) (type default) (color 0 0 0 0))
   )
+  (wire (pts (xy 102.616 56.388) (xy 110.744 56.388))
+    (stroke (width 0) (type default) (color 0 0 0 0))
+  )
   (wire (pts (xy 140.462 96.266) (xy 149.098 96.266))
     (stroke (width 0) (type default) (color 0 0 0 0))
@@
     (stroke (width 0) (type default) (color 0 0 0 0))
   )
+  (wire (pts (xy 45.72 106.426) (xy 64.008 106.426))
+    (stroke (width 0) (type default) (color 0 0 0 0))
+  )
   (wire (pts (xy 161.29 110.236) (xy 166.116 110.236))
     (stroke (width 0) (type default) (color 0 0 0 0))
@@
   )
   (wire (pts (xy 80.772 49.784) (xy 80.772 52.832))
+    (stroke (width 0) (type default) (color 0 0 0 0))
+  )
+  (wire (pts (xy 102.616 46.228) (xy 102.616 56.388))
     (stroke (width 0) (type default) (color 0 0 0 0))
   )
@@
     (pin "1")
   )
-  (symbol (lib_id "Connector:Conn_01x02_Male") (at 98.298 41.656 0) (unit 1)
-    (in_bom yes) (on_board yes)
-    (property "Reference" "J13" (id 0) (at 99.822 37.084 0))
-    (property "Value" "Alim 9V" (id 1) (at 99.822 38.862 0))
-    (property "Footprint" "Connector_PinHeader_2.54mm:PinHeader_1x02_P2.54mm_Vertical" (id 2) (at 98.298 41.656 0)
-      (effects (font (size 1.27 1.27)) hide)
-    )
-    (property "Datasheet" "~" (id 3) (at 98.298 41.656 0)
+  (symbol (lib_id "Connector:Conn_01x02_Male") (at 97.536 43.688 0) (unit 1)
+    (in_bom yes) (on_board yes)
+    (property "Reference" "J13" (id 0) (at 99.06 39.116 0))
+    (property "Value" "Alim 9V" (id 1) (at 99.06 40.894 0))
+    (property "Footprint" "Connector_PinHeader_2.54mm:PinHeader_1x02_P2.54mm_Vertical" (id 2) (at 97.536 43.688 0)
+      (effects (font (size 1.27 1.27)) hide)
+    )
+    (property "Datasheet" "~" (id 3) (at 97.536 43.688 0)
       (effects (font (size 1.27 1.27)) hide)
     )
@@
     (pin "1")
   )
-  (symbol (lib_id "Connector:Conn_01x02_Male") (at 33.274 93.726 0) (unit 1)
-    (in_bom yes) (on_board yes)
-    (property "Reference" "J12" (id 0) (at 36.068 89.662 0))
-    (property "Value" "Alim 6V" (id 1) (at 36.068 91.186 0))
-    (property "Footprint" "Connector_PinHeader_2.54mm:PinHeader_1x02_P2.54mm_Vertical" (id 2) (at 33.274 93.726 0)
-      (effects (font (size 1.27 1.27)) hide)
-    )
-    (property "Datasheet" "~" (id 3) (at 33.274 93.726 0)
-      (effects (font (size 1.27 1.27)) hide)
-    )
+  (symbol (lib_id "Connector:Conn_01x02_Male") (at 40.64 96.266 0) (unit 1)
+    (in_bom yes) (on_board yes)
+    (property "Reference" "J12" (id 0) (at 43.434 92.202 0))
+    (property "Value" "Alim 6V" (id 1) (at 43.434 93.726 0))
+    (property "Footprint" "Connector_PinHeader_2.54mm:PinHeader_1x02_P2.54mm_Vertical" (id 2) (at 40.64 96.266 0)
+      (effects (font (size 1.27 1.27)) hide)
+    )
+    (property "Datasheet" "~" (id 3) (at 40.64 96.266 0)
+      (effects (font (size 1.27 1.27)) hide)
+    )

Commit message: 1.6
Parts:
- renumbered J12 to J1, J13 to J2, J1 to J3, J2 to J4, J3 to J5, J4 to J6
Changed lines of the file:
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@@
   (symbol (lib_id "Connector:Conn_01x02_Male") (at 97.536 43.688 0) (unit 1)
     (in_bom yes) (on_board yes)
-    (property "Reference" "J13" (id 0) (at 99.06 39.116 0))
+    (property "Reference" "J2" (id 0) (at 99.06 39.116 0))
     (property "Value" "Alim 9V" (id 1) (at 99.06 40.894 0))
     (property "Footprint" "Connector_PinHeader_2.54mm:PinHeader_1x02_P2.54mm_Vertical" (id 2) (at 97.536 43.688 0)
@@
   (symbol (lib_id "Connector:Conn_01x02_Male") (at 171.196 107.188 180) (unit 1)
     (in_bom yes) (on_board yes)
-    (property "Reference" "J2" (id 0) (at 172.212 104.6479 0)
+    (property "Reference" "J4" (id 0) (at 172.212 104.6479 0)
       (effects (font (size 1.27 1.27)) (justify right))
     )
@@
   (symbol (lib_id "Connector:Conn_01x20_Female") (at 234.188 106.426 0) (unit 1)
     (in_bom yes) (on_board yes)
-    (property "Reference" "J4" (id 0) (at 235.966 106.4259 0)
+    (property "Reference" "J6" (id 0) (at 235.966 106.4259 0)
       (effects (font (size 1.27 1.27)) (justify left))
     )
@@
   (symbol (lib_id "Connector:Conn_01x20_Female") (at 205.232 106.426 0) (unit 1)
     (in_bom yes) (on_board yes) (fields_autoplaced)
-    (property "Reference" "J3" (id 0) (at 206.756 106.4259 0)
+    (property "Reference" "J5" (id 0) (at 206.756 106.4259 0)
       (effects (font (size 1.27 1.27)) (justify left))
     )
@@
   (symbol (lib_id "Connector:Conn_01x02_Male") (at 104.902 107.188 180) (unit 1)
     (in_bom yes) (on_board yes)
-    (property "Reference" "J1" (id 0) (at 105.918 104.6479 0)
+    (property "Reference" "J3" (id 0) (at 105.918 104.6479 0)
       (effects (font (size 1.27 1.27)) (justify right))
     )
@@
   (symbol (lib_id "Connector:Conn_01x02_Male") (at 40.64 96.266 0) (unit 1)
     (in_bom yes) (on_board yes)
-    (property "Reference" "J12" (id 0) (at 43.434 92.202 0))
+    (property "Reference" "J1" (id 0) (at 43.434 92.202 0))
     (property "Value" "Alim 6V" (id 1) (at 43.434 93.726 0))
     (property "Footprint" "Connector_PinHeader_2.54mm:PinHeader_1x02_P2.54mm_Vertical" (id 2) (at 40.64 96.266 0)

Commit message: 2.0 alabama
Parts:
- added J14, J15: 01x20_Female, Connector_PinSocket_2.54mm:PinSocket_1x20_P2.54mm_Vertical, symbol Connector:Conn_01x20_Female
Connections:
- net 3.3V: now also J14.9 (Pin_9), J15.10 (Pin_10)
- net 5V: now also J14.11 (Pin_11)
- net GND: now also J14.10 (Pin_10), J14.12 (Pin_12), J15.9 (Pin_9)
- net P0: now also J15.1 (Pin_1)
- net P1: now also J15.2 (Pin_2)
- net P10: now also J15.15 (Pin_15)
- net P11: now also J15.16 (Pin_16)
- net P12: now also J15.17 (Pin_17)
- net P13: now also J15.18 (Pin_18)
- net P14: now also J15.19 (Pin_19)
- net P15: now also J15.20 (Pin_20)
- net P16: now also J14.20 (Pin_20)
- net P17: now also J14.19 (Pin_19)
- net P18: now also J14.18 (Pin_18)
- net P19: now also J14.17 (Pin_17)
- net P2: now also J15.3 (Pin_3)
- net P20: now also J14.16 (Pin_16)
- net P21: now also J14.15 (Pin_15)
- net P22: now also J14.14 (Pin_14)
- net P23: now also J14.13 (Pin_13)
- net P24: now also J14.8 (Pin_8)
- net P25: now also J14.7 (Pin_7)
- net P26: now also J14.6 (Pin_6)
- net P27: now also J14.5 (Pin_5)
- net P28_SCL: now also J14.4 (Pin_4)
- net P29_SDA: now also J14.3 (Pin_3)
- net P3: now also J15.4 (Pin_4)
- net P30_TX: now also J14.2 (Pin_2)
- net P31_RX: now also J14.1 (Pin_1)
- net P4: now also J15.5 (Pin_5)
- net P5: now also J15.6 (Pin_6)
- net P6: now also J15.7 (Pin_7)
- net P7: now also J15.8 (Pin_8)
- net P8: now also J15.13 (Pin_13)
- net P9: now also J15.14 (Pin_14)
- net RESET: now also J15.11 (Pin_11)

Commit message: 2.1 Missouri
Parts:
- added J12, J13, J16, J17: Conn_01x03_Male, Connector_PinHeader_2.54mm:PinHeader_1x03_P2.54mm_Vertical, symbol Connector:Conn_01x03_Male
Connections:
- net 3.3V: now also J12.1 (Pin_1), J13.1 (Pin_1), J16.1 (Pin_1), J17.1 (Pin_1)
- net GND: now also J12.2 (Pin_2), J13.2 (Pin_2), J16.2 (Pin_2), J17.2 (Pin_2)
- net P4: now also J12.3 (Pin_3)
- net P5: now also J13.3 (Pin_3)
- net P6: now also J16.3 (Pin_3)
- net P7: now also J17.3 (Pin_3)
Changed lines of the file:
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@@
     (effects (font (size 1.27 1.27)) (justify right bottom))
+  )
+  (label "P7" (at 265.176 129.286 0)
+    (effects (font (size 1.27 1.27)) (justify left bottom))
   )
   (label "6V" (at 133.096 76.454 0)
@@
     (effects (font (size 1.27 1.27)) (justify left bottom))
   )
+  (label "GND" (at 265.176 95.758 0)
+    (effects (font (size 1.27 1.27)) (justify left bottom))
+  )
   (label "9V" (at 80.772 49.784 180)
     (effects (font (size 1.27 1.27)) (justify right bottom))
@@
     (effects (font (size 1.27 1.27)) (justify right bottom))
   )
+  (label "GND" (at 265.176 106.172 0)
+    (effects (font (size 1.27 1.27)) (justify left bottom))
+  )
   (label "P20" (at 199.898 68.326 180)
     (effects (font (size 1.27 1.27)) (justify right bottom))
@@
     (effects (font (size 1.27 1.27)) (justify right bottom))
   )
+  (label "P6" (at 265.176 118.872 0)
+    (effects (font (size 1.27 1.27)) (justify left bottom))
+  )
   (label "P5" (at 228.854 42.926 180)
     (effects (font (size 1.27 1.27)) (justify right bottom))
@@
     (effects (font (size 1.27 1.27)) (justify right bottom))
   )
+  (label "GND" (at 265.176 126.746 0)
+    (effects (font (size 1.27 1.27)) (justify left bottom))
+  )
   (label "P18" (at 200.152 126.746 180)
     (effects (font (size 1.27 1.27)) (justify right bottom))
@@
     (effects (font (size 1.27 1.27)) (justify right bottom))
   )
+  (label "GND" (at 265.176 116.332 0)
+    (effects (font (size 1.27 1.27)) (justify left bottom))
+  )
   (label "P2" (at 120.142 98.806 180)
     (effects (font (size 1.27 1.27)) (justify right bottom))
   )
+  (label "3.3V" (at 265.176 103.632 0)
+    (effects (font (size 1.27 1.27)) (justify left bottom))
+  )
   (label "3.3V" (at 228.854 53.086 180)
     (effects (font (size 1.27 1.27)) (justify right bottom))
   )
+  (label "P5" (at 265.176 108.712 0)
+    (effects (font (size 1.27 1.27)) (justify left bottom))
+  )
   (label "6V" (at 70.866 49.784 180)
     (effects (font (size 1.27 1.27)) (justify right bottom))
@@
     (effects (font (size 1.27 1.27)) (justify right bottom))
   )
+  (label "P4" (at 265.176 98.298 0)
+    (effects (font (size 1.27 1.27)) (justify left bottom))
+  )
   (label "P0" (at 228.854 30.226 180)
     (effects (font (size 1.27 1.27)) (justify right bottom))
@@
     (effects (font (size 1.27 1.27)) (justify right bottom))
   )
+  (label "3.3V" (at 265.176 124.206 0)
+    (effects (font (size 1.27 1.27)) (justify left bottom))
+  )
   (label "P4" (at 228.854 40.386 180)
     (effects (font (size 1.27 1.27)) (justify right bottom))
@@
     (effects (font (size 1.27 1.27)) (justify right bottom))
   )
+  (label "3.3V" (at 265.176 113.792 0)
+    (effects (font (size 1.27 1.27)) (justify left bottom))
+  )
   (label "P25" (at 199.898 45.466 180)
     (effects (font (size 1.27 1.27)) (justify right bottom))
+  )
+  (label "3.3V" (at 265.176 93.218 0)
+    (effects (font (size 1.27 1.27)) (justify left bottom))
   )
   (label "P7" (at 229.108 101.346 180)
@@
     (pin "1")
   )
+  (symbol (lib_id "Connector:Conn_01x03_Male") (at 260.096 106.172 0) (unit 1)
+    (in_bom yes) (on_board yes)
+    (property "Reference" "J13" (id 0) (at 262.89 99.822 0))
+    (property "Value" "Conn_01x03_Male" (id 1) (at 260.731 101.346 0))
+    (property "Footprint" "Connector_PinHeader_2.54mm:PinHeader_1x03_P2.54mm_Vertical" (id 2) (at 260.096 106.172 0)
+      (effects (font (size 1.27 1.27)) hide)
+    )
+    (property "Datasheet" "~" (id 3) (at 260.096 106.172 0)
+      (effects (font (size 1.27 1.27)) hide)
+    )
+    (pin "1")
+    (pin "2")
+    (pin "3")
+  )
+  (symbol (lib_id "Connector:Conn_01x03_Male") (at 260.096 95.758 0) (unit 1)
+    (in_bom yes) (on_board yes)
+    (property "Reference" "J12" (id 0) (at 262.89 89.408 0))
+    (property "Value" "Conn_01x03_Male" (id 1) (at 260.731 90.932 0))
+    (property "Footprint" "Connector_PinHeader_2.54mm:PinHeader_1x03_P2.54mm_Vertical" (id 2) (at 260.096 95.758 0)
+      (effects (font (size 1.27 1.27)) hide)
+    )
+    (property "Datasheet" "~" (id 3) (at 260.096 95.758 0)
+      (effects (font (size 1.27 1.27)) hide)
+    )
+    (pin "1")
+    (pin "2")
+    (pin "3")
+  )
   (symbol (lib_id "power:GND") (at 158.496 56.388 0) (unit 1)
     (in_bom yes) (on_board yes) (fields_autoplaced)
@@
     (pin "1")
     (pin "2")
+  )
+  (symbol (lib_id "Connector:Conn_01x03_Male") (at 260.096 126.746 0) (unit 1)
+    (in_bom yes) (on_board yes)
+    (property "Reference" "J17" (id 0) (at 262.89 120.396 0))
+    (property "Value" "Conn_01x03_Male" (id 1) (at 260.731 121.92 0))
+    (property "Footprint" "Connector_PinHeader_2.54mm:PinHeader_1x03_P2.54mm_Vertical" (id 2) (at 260.096 126.746 0)
+      (effects (font (size 1.27 1.27)) hide)
+    )
+    (property "Datasheet" "~" (id 3) (at 260.096 126.746 0)
+      (effects (font (size 1.27 1.27)) hide)
+    )
+    (pin "1")
+    (pin "2")
+    (pin "3")
   )
   (symbol (lib_id "Projet2_LibraryCustom:MC33269DR2-5.0G") (at 125.984 43.688 0) (unit 1)
@@
     (pin "2")
   )
+  (symbol (lib_id "Connector:Conn_01x03_Male") (at 260.096 116.332 0) (unit 1)
+    (in_bom yes) (on_board yes)
+    (property "Reference" "J16" (id 0) (at 262.89 109.982 0))
+    (property "Value" "Conn_01x03_Male" (id 1) (at 260.731 111.506 0))
+    (property "Footprint" "Connector_PinHeader_2.54mm:PinHeader_1x03_P2.54mm_Vertical" (id 2) (at 260.096 116.332 0)
+      (effects (font (size 1.27 1.27)) hide)
+    )
+    (property "Datasheet" "~" (id 3) (at 260.096 116.332 0)
+      (effects (font (size 1.27 1.27)) hide)
+    )
+    (pin "1")
+    (pin "2")
+    (pin "3")
+  )
   (symbol (lib_id "Connector:Conn_01x20_Female") (at 205.232 106.426 0) (unit 1)
