File: PCB/Carte Mere/untitled.kicad_sch (KiCad schematic)
At the start: 35 parts, among them J1 Alim 6V, J12 Conn_01x03_Male, J13 Conn_01x03_Male, J14 01x20_Female, J15 01x20_Female, J16 Conn_01x03_Male, J17 Conn_01x03_Male, J2 Alim 9V, J3 Moteur, J4 Moteur, J5 01x20_Female, J6 01x20_Female, U1 ZXBM5210-S, U2 MC33269DR2-5.0G, U3 ZXBM5210-S, U4 LD1117S33TR_SOT223

Commit message: 2.2 Florida
Parts:
- J12, J13, J16, J17: value Conn_01x03_Male -> Conn_Tcrt5000
Connections:
- no-connect marks 0 -> 2
Changed lines of the file:
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@@
   (junction (at 166.116 110.236) (diameter 0) (color 0 0 0 0)
   )
+  (no_connect (at 228.854 58.166))
+  (no_connect (at 229.108 111.506))
   (wire (pts (xy 166.116 101.6) (xy 166.116 104.648))
     (stroke (width 0) (type default) (color 0 0 0 0))
@@
     (stroke (width 0) (type default) (color 0 0 0 0))
   )
-  (label "3.3V" (at 229.108 106.426 180)
-    (effects (font (size 1.27 1.27)) (justify right bottom))
-  )
   (label "P12" (at 228.854 70.866 180)
     (effects (font (size 1.27 1.27)) (justify right bottom))
@@
     (effects (font (size 1.27 1.27)) (justify right bottom))
   )
-  (label "3.3V" (at 200.152 103.886 180)
-    (effects (font (size 1.27 1.27)) (justify right bottom))
-  )
   (label "GND" (at 199.898 53.086 180)
     (effects (font (size 1.27 1.27)) (justify right bottom))
@@
     (effects (font (size 1.27 1.27)) (justify right bottom))
   )
-  (label "P8" (at 229.108 114.046 180)
-    (effects (font (size 1.27 1.27)) (justify right bottom))
-  )
   (label "P3" (at 120.142 101.346 180)
     (effects (font (size 1.27 1.27)) (justify right bottom))
@@
   (label "P7" (at 228.854 48.006 180)
     (effects (font (size 1.27 1.27)) (justify right bottom))
+  )
+  (global_label "P8" (shape input) (at 229.108 114.046 180) (fields_autoplaced)
+    (effects (font (size 1.27 1.27)) (justify right))
+    (property "Intersheet References" "${INTERSHEET_REFS}" (id 0) (at 224.2154 113.9666 0)
+      (effects (font (size 1.27 1.27)) (justify right) hide)
+    )
+  )
+  (global_label "3.3V" (shape input) (at 229.108 106.426 180) (fields_autoplaced)
+    (effects (font (size 1.27 1.27)) (justify right))
+    (property "Intersheet References" "${INTERSHEET_REFS}" (id 0) (at 222.5825 106.3466 0)
+      (effects (font (size 1.27 1.27)) (justify right) hide)
+    )
+  )
+  (global_label "3.3V" (shape input) (at 200.152 103.886 180) (fields_autoplaced)
+    (effects (font (size 1.27 1.27)) (justify right))
+    (property "Intersheet References" "${INTERSHEET_REFS}" (id 0) (at 193.6265 103.8066 0)
+      (effects (font (size 1.27 1.27)) (justify right) hide)
+    )
   )
   (symbol (lib_id "Device:C") (at 53.848 76.454 270) (unit 1)
@@
   (symbol (lib_id "Connector:Conn_01x03_Male") (at 260.096 106.172 0) (unit 1)
     (in_bom yes) (on_board yes)
-    (property "Reference" "J13" (id 0) (at 262.89 99.822 0))
-    (property "Value" "Conn_01x03_Male" (id 1) (at 260.731 101.346 0))
+    (property "Reference" "J13" (id 0) (at 262.89 99.568 0))
+    (property "Value" "Conn_Tcrt5000" (id 1) (at 262.382 101.092 0))
     (property "Footprint" "Connector_PinHeader_2.54mm:PinHeader_1x03_P2.54mm_Vertical" (id 2) (at 260.096 106.172 0)
       (effects (font (size 1.27 1.27)) hide)
@@
   (symbol (lib_id "Connector:Conn_01x03_Male") (at 260.096 95.758 0) (unit 1)
     (in_bom yes) (on_board yes)
-    (property "Reference" "J12" (id 0) (at 262.89 89.408 0))
-    (property "Value" "Conn_01x03_Male" (id 1) (at 260.731 90.932 0))
+    (property "Reference" "J12" (id 0) (at 262.89 89.154 0))
+    (property "Value" "Conn_Tcrt5000" (id 1) (at 261.62 90.678 0))
     (property "Footprint" "Connector_PinHeader_2.54mm:PinHeader_1x03_P2.54mm_Vertical" (id 2) (at 260.096 95.758 0)
       (effects (font (size 1.27 1.27)) hide)
@@
   (symbol (lib_id "Connector:Conn_01x03_Male") (at 260.096 126.746 0) (unit 1)
     (in_bom yes) (on_board yes)
-    (property "Reference" "J17" (id 0) (at 262.89 120.396 0))
-    (property "Value" "Conn_01x03_Male" (id 1) (at 260.731 121.92 0))
+    (property "Reference" "J17" (id 0) (at 263.144 120.142 0))
+    (property "Value" "Conn_Tcrt5000" (id 1) (at 262.636 121.666 0))
     (property "Footprint" "Connector_PinHeader_2.54mm:PinHeader_1x03_P2.54mm_Vertical" (id 2) (at 260.096 126.746 0)
       (effects (font (size 1.27 1.27)) hide)
@@
   (symbol (lib_id "Connector:Conn_01x03_Male") (at 260.096 116.332 0) (unit 1)
     (in_bom yes) (on_board yes)
-    (property "Reference" "J16" (id 0) (at 262.89 109.982 0))
-    (property "Value" "Conn_01x03_Male" (id 1) (at 260.731 111.506 0))
+    (property "Reference" "J16" (id 0) (at 262.89 109.728 0))
+    (property "Value" "Conn_Tcrt5000" (id 1) (at 262.636 111.252 0))
     (property "Footprint" "Connector_PinHeader_2.54mm:PinHeader_1x03_P2.54mm_Vertical" (id 2) (at 260.096 116.332 0)
       (effects (font (size 1.27 1.27)) hide)
