File: PCB/Carte Mere/untitled.kicad_sch (KiCad schematic)
At the start: 35 parts, among them J1 Alim 6V, J12 Conn_Tcrt5000, J13 Conn_Tcrt5000, J14 01x20_Female, J15 01x20_Female, J16 Conn_Tcrt5000, J17 Conn_Tcrt5000, J2 Alim 9V, J3 Moteur, J4 Moteur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

Commit message: Fixed Zach's errors :/ smh
Changed lines of the file:
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@@
   (junction (at 149.098 101.6) (diameter 0) (color 0 0 0 0)
+  )
+  (junction (at 142.24 43.688) (diameter 0) (color 0 0 0 0)
   )
   (junction (at 144.526 43.688) (diameter 0) (color 0 0 0 0)
@@
     (stroke (width 0) (type default) (color 0 0 0 0))
   )
-  (wire (pts (xy 138.684 43.688) (xy 144.526 43.688))
+  (wire (pts (xy 138.684 43.688) (xy 142.24 43.688))
     (stroke (width 0) (type default) (color 0 0 0 0))
   )
   (wire (pts (xy 86.614 119.126) (xy 94.996 119.126))
+    (stroke (width 0) (type default) (color 0 0 0 0))
+  )
+  (wire (pts (xy 142.24 43.688) (xy 144.526 43.688))
     (stroke (width 0) (type default) (color 0 0 0 0))
   )
@@
     (pin "8")
   )
+  (symbol (lib_id "power:PWR_FLAG") (at 142.24 43.688 0) (unit 1)
+    (in_bom yes) (on_board yes) (fields_autoplaced)
+    (property "Reference" "#FLG0101" (id 0) (at 142.24 41.783 0)
+      (effects (font (size 1.27 1.27)) hide)
+    )
+    (property "Value" "PWR_FLAG" (id 1) (at 142.24 38.354 0))
+    (property "Footprint" "" (id 2) (at 142.24 43.688 0)
+      (effects (font (size 1.27 1.27)) hide)
+    )
+    (property "Datasheet" "~" (id 3) (at 142.24 43.688 0)
+      (effects (font (size 1.27 1.27)) hide)
+    )
+    (pin "1")
+  )
   (symbol (lib_id "Device:LED") (at 82.804 105.41 90) (unit 1)
