File: PCB/PowerSupply/PowerSupply/PowerSupply.kicad_pcb (KiCad board)
At the start: 2 copper layers, 38 parts, among them J1 Vin, J2 Vout, J3 Vin, J4 Vout, J5 Vout, J6 Vout, Q1 CSD16301Q2, Q2 CSD16301Q2, U3 LM3478MM, U4 LM3478MM

Commit message: Finished v0.1
Parts:
- moved J6 8.76 mm to (47.5, 43.5)
- moved J2 3.68 mm to (47.5, 47.1)
- moved L1 0.76 mm to (29.0, 53.8)
- moved L2 0.75 mm to (29.0, 32.3)
Connections:
- C1 pad 1: GND -> Net-(C1-Pad1)
- D1 pad 1: GND -> Net-(C1-Pad1)
- J2 pad 1: GND -> Net-(C1-Pad1)
- J6 pad 1: GND -> Net-(C1-Pad1)
- R2 pad 2: GND -> Net-(C1-Pad1)
Routing:
- net Net-(C1-Pad1): track 0.00 -> 31.5 mm
- net GND: track 176.5 -> 145.3 mm, vias 1 -> 0
- net Net-(D1-Pad2): track 19.7 -> 33.3 mm, vias 0 -> 2
- net Net-(D2-Pad2): track 19.7 -> 33.1 mm, vias 0 -> 2
- net Net-(Cbyp2-Pad1): track 19.3 -> 20.3 mm
